File: KiCAD Files/OpenHAK_03.sch (KiCad schematic (older format))
At the start: 40 parts, among them P1 M50-3140845, P2 USB_OTG, U1 rfd_77101, U2 MAX30100, U3 MIC5365-1.8YMT-TZ, U4 BMI160, U5 MCP73831T-2ATI/OT, U6 MIC5365-3.0YMT-TZ, U7 TXS0102DQER, U8 MAX809SQ308T1G

Commit message: removed some stuff we don't need and made notes about changes to pcb
Parts:
- removed U8: MAX809SQ308T1G, TO_SOT_Packages_SMD:SOT-323_SC-70, symbol OpenHAK_03:MAX809
- C14: value 1uF -> 0.1uF
Connections:
- net labels removed: EN
- wire segments 218 -> 216
Other:
- note added: "Add two more breakouts here"
- note removed: "Change pullup connection to VDD"
- note removed: "This voltage trigger\nmight not be necessary…"
- moved on the sheet: C10, C14, R7, R8
