File: KiCAD Files/OpenHAK_03.sch (KiCad schematic (older format))
At the start: 40 parts, among them P1 M50-3140845, P2 USB_OTG, U1 rfd_77101, U2 MAX30100, U3 MIC5365-1.8YMT-TZ, U4 BMI160, U5 MCP73831T-2ATI/OT, U6 MIC5365-3.0YMT-TZ, U7 TXS0102DQER, U8 MAX809SQ308T1G

Commit message: Major changes to the board layout
took some things off, put some things on, and moved some things around
Parts:
- removed U8: MAX809SQ308T1G, TO_SOT_Packages_SMD:SOT-323_SC-70, symbol OpenHAK_03:MAX809
- BT1: symbol OpenHAK_03:Battery -> OpenHAK_03:OpenHAK_03_Battery
- D1: symbol OpenHAK_03:Led_RGB_CA -> OpenHAK_03:OpenHAK_03_Led_RGB_CA
- D3: symbol OpenHAK_03:Dialight_R_G_LED -> OpenHAK_03:OpenHAK_03_Dialight_R_G_LED
- P1: value M50-3140845 -> Harwin M52 Series; footprint Solutions:M50-3140845_1x8_SMT_F -> Solutions:M52-Series_Harwin_SMT_10P; symbol Connector_Generic:Conn_01x08 -> Connector:Conn_01x10_Female
- U1: symbol OpenHAK_03:rfd_77101 -> OpenHAK_03:OpenHAK_03_rfd_77101
- U2: symbol OpenHAK_03:MAX30100 -> OpenHAK_03:OpenHAK_03_MAX30100
- U3, U6: symbol OpenHAK_03:MIC5365-X.XYMT-TZ -> OpenHAK_03:OpenHAK_03_MIC5365-X.XYMT-TZ
- U4: symbol OpenHAK_03:BMI160 -> OpenHAK_03:OpenHAK_03_BMI160
- U5: symbol OpenHAK_03:MCP73831 -> OpenHAK_03:OpenHAK_03_MCP73831
- U7: symbol OpenHAK_03:TXS0102_LEVEL_SHIFTER_X2SON8 -> OpenHAK_03:OpenHAK_03_TXS0102_LEVEL_SHIFTER_X2SON8
Connections:
- net labels added: PIN_21, PIN_24, V_BATT
- net labels removed: EN
- wire segments 218 -> 217
Other:
- note added: "move away from corner?"
- note removed: "Change pullup connection to VDD"
- note removed: "This voltage trigger\nmight not be necessary…"
- moved on the sheet: C10, C14, R7, R8

Commit message: Cleaned up silk
Other:
- note added: "GPIO 3 / ANALOG 4\nGPIO 1 / ANALOG 2\nGPIO 2 / ANALOG 3\nGPIO 0 / AREF 0\nGPIO 25\nGPIO 24\nGPIO 21\n"
- note removed: "GPIO 3 / ANALOG 4\nGPIO 1 / ANALOG 2\nGPIO 2 / ANALOG 3\nGPIO 0 / AREF 0\nGPIO 25\n"
Changed lines of the file:
@@
 EESchema Schematic File Version 4
+LIBS:OpenHAK_03-cache
 EELAYER 26 0
 EELAYER END
@@
 Wire Wire Line
 	6050 2050 6200 2050
-Text Notes 7050 6050 0    60   ~ 0
-GPIO 3 / ANALOG 4\nGPIO 1 / ANALOG 2\nGPIO 2 / ANALOG 3\nGPIO 0 / AREF 0\nGPIO 25\n
+Text Notes 7050 6250 0    60   ~ 0
+GPIO 3 / ANALOG 4\nGPIO 1 / ANALOG 2\nGPIO 2 / ANALOG 3\nGPIO 0 / AREF 0\nGPIO 25\nGPIO 24\nGPIO 21\n
 Wire Wire Line
 	1900 1350 1900 1400
