File: KiCAD Files/OpenHAK_03.sch (KiCad schematic (older format))
At the start: 39 parts, among them P1 Harwin M52 Series, P2 USB_OTG, U1 rfd_77101, U2 MAX30100, U3 MIC5365-1.8YMT-TZ, U4 BMI160, U5 MCP73831T-2ATI/OT, U6 MIC5365-3.0YMT-TZ, U7 TXS0102DQER

Commit message: generated gerbers and polished bom
Connections:
- wire segments 217 -> 215
Changed lines of the file:
@@
 EESchema Schematic File Version 4
+LIBS:OpenHAK_03-cache
 EELAYER 26 0
 EELAYER END
@@
 L power:VDD #PWR06
 U 1 1 57CDC75F
-P 7350 1050
-F 0 "#PWR06" H 7350 900 50  0001 C CNN
-F 1 "VDD" H 7350 1200 50  0000 C CNN
-F 2 "" H 7350 1050 50  0000 C CNN
-F 3 "" H 7350 1050 50  0000 C CNN
-	1    7350 1050
+P 7500 1050
+F 0 "#PWR06" H 7500 900 50  0001 C CNN
+F 1 "VDD" H 7500 1200 50  0000 C CNN
+F 2 "" H 7500 1050 50  0000 C CNN
+F 3 "" H 7500 1050 50  0000 C CNN
+	1    7500 1050
 	1    0    0    -1
 $EndComp
@@
 Connection ~ 5950 7300
 Wire Wire Line
-	7350 1150 7350 1050
+	7500 1150 7500 1050
 Wire Wire Line
 	5500 1150 5600 1150
@@
 Wire Wire Line
 	7500 1150 7500 1200
-Connection ~ 7350 1150
+Connection ~ 7500 1150
 Wire Wire Line
 	7500 1550 7500 1500
@@
 Connection ~ 1900 2200
 Wire Wire Line
-	5600 2050 5750 2050
-Wire Wire Line
-	5600 2050 5600 2000
+	5750 2050 5750 1950
 Wire Wire Line
 	5750 2100 5750 2050
@@
 	5950 7300 5950 7550
 Wire Wire Line
-	7350 1150 7500 1150
-Wire Wire Line
 	5600 1150 5750 1150
 Wire Wire Line
@@
 $EndComp
 Wire Wire Line
-	7050 1150 7350 1150
+	7050 1150 7500 1150
 Wire Wire Line
 	7050 1250 7200 1250
@@
 L power:VDD #PWR0101
 U 1 1 5C75E84A
-P 5600 2000
-F 0 "#PWR0101" H 5600 1850 50  0001 C CNN
-F 1 "VDD" H 5600 2150 50  0000 C CNN
-F 2 "" H 5600 2000 50  0000 C CNN
-F 3 "" H 5600 2000 50  0000 C CNN
-	1    5600 2000
-	1    0    0    -1
-$EndComp
+P 5750 1950
+F 0 "#PWR0101" H 5750 1800 50  0001 C CNN
+F 1 "VDD" H 5750 2100 50  0000 C CNN
+F 2 "" H 5750 1950 50  0000 C CNN
+F 3 "" H 5750 1950 50  0000 C CNN
+	1    5750 1950
+	1    0    0    -1
+$EndComp
