File: KiCAD Files/OpenHAK_03.kicad_pcb (KiCad board)
At the start: 4 copper layers, 38.1 x 25.4 mm, 52 parts, among them P1 Harwin M52 Series, P2 USB_OTG, U1 rfd_77101, U2 MAX30100, U3 MIC5365-1.8YMT-TZ, U4 BMI160, U5 MCP73831T-2ATI/OT, U6 MIC5365-3.0YMT-TZ, U7 TXS0102DQER

Commit message: Cleaned up silk
Parts:
- removed G***: LOGO, Solutions:BHVsmall
Other:
- board text added: "pithy motto"
- board text removed: "BioHacking Village"
- board text removed: "DEFCON24"
